Commit message: add ex05

File: Lab_5/ex05/my_robot-main/robot_description/urdf/gazebo.urdf.xacro (robot description, xacro)
@@ -30,5 +30,5 @@
             <child_frame_id>robot/base_link</child_frame_id>
             <wheel_separation>0.291</wheel_separation>
-            <wheel_radius>0.0495</wheel_radius>
+            <wheel_radius>0.1</wheel_radius>
             <odom_publish_frequency>10</odom_publish_frequency>
         </plugin>

File: Lab_5/ex05/my_robot-main/robot_description/urdf/robot.urdf.xacro (robot description, xacro)
@@ -13,5 +13,5 @@
     <xacro:property name="petal_radius" value="0.2"/>
     <xacro:property name="petal_height" value="0.05"/>
-    <xacro:property name="wheel_radius" value="0.0495"/>
+    <xacro:property name="wheel_radius" value="0.1"/>
     <xacro:property name="wheel_thickness" value="0.039"/>
     <xacro:property name="wheel_mass" value="0.075"/>
@@ -221,12 +221,4 @@
         </geometry>
     </collision>
-    <inertial>
-        <!-- Параметры инерции для stem -->
-        <origin xyz="0 0 0.05" rpy="0 0 0"/>
-        <mass value="${mass}" />
-        <inertia ixx="1e-6" ixy="0.0" ixz="0.0"
-                 iyy="1e-6" iyz="0.0"
-                 izz="1e-6" />
-    </inertial>
     </link>
     <gazebo reference="stem">
@@ -250,12 +242,4 @@
         </geometry>
     </collision>
-    <inertial>
-        <!-- Параметры инерции для stem -->
-        <origin xyz="0 0 0.05" rpy="0 0 0"/>
-        <mass value="${mass}" />
-        <inertia ixx="1e-6" ixy="0.0" ixz="0.0"
-                 iyy="1e-6" iyz="0.0"
-                 izz="1e-6" />
-    </inertial>
     </link>
     <gazebo reference="flower_disk">
@@ -267,10 +251,10 @@
     	<child link="petal_one"/>
     	<axis xyz="0 0 1"/>
- 	<origin rpy="0 -0.3 0" xyz="0.4 0 0.05"/>
+ 	<origin rpy="0 -0.4 0" xyz="0.4 0 0.08"/>
     </joint>
     <link name="petal_one">
     <visual>
         <geometry>
-            <cylinder radius="${petal_radius}" length="${petal_height}"/> <!-- Измените параметры, если необходимо -->
+            <cylinder radius="${petal_radius}" length="${petal_height/4}"/> <!-- Измените параметры, если необходимо -->
         </geometry>
         <material name="white"/>
@@ -278,15 +262,7 @@
     <collision>
         <geometry>
-            <cylinder radius="${petal_radius}" length="${petal_height}"/>
-        </geometry>
-    </collision>
-    <inertial>
-        <!-- Параметры инерции для stem -->
-        <origin xyz="0 0 0.05" rpy="0 0 0"/>
-        <mass value="0" />
-        <inertia ixx="1e-6" ixy="0.0" ixz="0.0"
-                 iyy="1e-6" iyz="0.0"
-                 izz="1e-6" />
-    </inertial>
+            <cylinder radius="${petal_radius}" length="${petal_height/4}"/>
+        </geometry>
+    </collision>
     </link>
     <gazebo reference="petal_one">
@@ -298,10 +274,10 @@
     	<child link="petal_two"/>
     	<axis xyz="0 0 1"/>
- 	<origin rpy="0 0.3 0" xyz="-0.4 0 0.05"/>
+ 	<origin rpy="0 0.4 0" xyz="-0.4 0 0.08"/>
     </joint>
     <link name="petal_two">
     <visual>
         <geometry>
-            <cylinder radius="${petal_radius}" length="${petal_height}"/> <!-- Измените параметры, если необходимо -->
+            <cylinder radius="${petal_radius}" length="${petal_height/4}"/> <!-- Измените параметры, если необходимо -->
         </geometry>
         <material name="white"/>
@@ -309,15 +285,7 @@
     <collision>
         <geometry>
-            <cylinder radius="${petal_radius}" length="${petal_height}"/>
-        </geometry>
-    </collision>
-    <inertial>
-        <!-- Параметры инерции для stem -->
-        <origin xyz="0 0 0.05" rpy="0 0 0"/>
-        <mass value="0" />
-        <inertia ixx="1e-6" ixy="0.0" ixz="0.0"
-                 iyy="1e-6" iyz="0.0"
-                 izz="1e-6" />
-    </inertial>
+            <cylinder radius="${petal_radius}" length="${petal_height/4}"/>
+        </geometry>
+    </collision>
     </link>
     <gazebo reference="petal_two">
@@ -329,10 +297,10 @@
     	<child link="petal_three"/>
     	<axis xyz="0 0 1"/>
- 	<origin rpy="0.3 0 0" xyz="0 0.4 0.05"/>
+ 	<origin rpy="0.4 0 0" xyz="0 0.4 0.08"/>
     </joint>
     <link name="petal_three">
     <visual>
         <geometry>
-            <cylinder radius="${petal_radius}" length="${petal_height}"/> <!-- Измените параметры, если необходимо -->
+            <cylinder radius="${petal_radius}" length="${petal_height/4}"/> <!-- Измените параметры, если необходимо -->
         </geometry>
         <material name="white"/>
@@ -340,15 +308,7 @@
     <collision>
         <geometry>
-            <cylinder radius="${petal_radius}" length="${petal_height}"/>
-        </geometry>
-    </collision>
-    <inertial>
-        <!-- Параметры инерции для stem -->
-        <origin xyz="0 0 0.05" rpy="0 0 0"/>
-        <mass value="0" />
-        <inertia ixx="1e-6" ixy="0.0" ixz="0.0"
-                 iyy="1e-6" iyz="0.0"
-                 izz="1e-6" />
-    </inertial>
+            <cylinder radius="${petal_radius}" length="${petal_height/4}"/>
+        </geometry>
+    </collision>
     </link>
     <gazebo reference="petal_three">
@@ -360,10 +320,10 @@
     	<child link="petal_four"/>
     	<axis xyz="0 0 1"/>
- 	<origin rpy="0.2 -0.2 0" xyz="0.3 0.3 0.05"/>
+ 	<origin rpy="0.3 -0.3 0" xyz="0.3 0.3 0.08"/>
     </joint>
     <link name="petal_four">
     <visual>
         <geometry>
-            <cylinder radius="${petal_radius}" length="${petal_height}"/> <!-- Измените параметры, если необходимо -->
+            <cylinder radius="${petal_radius}" length="${petal_height/4}"/> <!-- Измените параметры, если необходимо -->
         </geometry>
         <material name="orange"/>
@@ -371,15 +331,7 @@
     <collision>
         <geometry>
-            <cylinder radius="${petal_radius}" length="${petal_height}"/>
-        </geometry>
-    </collision>
-    <inertial>
-        <!-- Параметры инерции для stem -->
-        <origin xyz="0 0 0.05" rpy="0 0 0"/>
-        <mass value="0" />
-        <inertia ixx="1e-6" ixy="0.0" ixz="0.0"
-                 iyy="1e-6" iyz="0.0"
-                 izz="1e-6" />
-    </inertial>
+            <cylinder radius="${petal_radius}" length="${petal_height/4}"/>
+        </geometry>
+    </collision>
     </link>
     <gazebo reference="petal_four">
@@ -391,10 +343,10 @@
     	<child link="petal_five"/>
     	<axis xyz="0 0 1"/>
- 	<origin rpy="-0.3 0 0" xyz="0 -0.4 0.05"/>
+ 	<origin rpy="-0.4 0 0" xyz="0 -0.4 0.08"/>
     </joint>
     <link name="petal_five">
     <visual>
         <geometry>
-            <cylinder radius="${petal_radius}" length="${petal_height}"/> <!-- Измените параметры, если необходимо -->
+            <cylinder radius="${petal_radius}" length="${petal_height/4}"/> <!-- Измените параметры, если необходимо -->
         </geometry>
         <material name="white"/>
@@ -402,15 +354,7 @@
     <collision>
         <geometry>
-            <cylinder radius="${petal_radius}" length="${petal_height}"/>
-        </geometry>
-    </collision>
-    <inertial>
-        <!-- Параметры инерции для stem -->
-        <origin xyz="0 0 0.05" rpy="0 0 0"/>
-        <mass value="0" />
-        <inertia ixx="1e-6" ixy="0.0" ixz="0.0"
-                 iyy="1e-6" iyz="0.0"
-                 izz="1e-6" />
-    </inertial>
+            <cylinder radius="${petal_radius}" length="${petal_height/4}"/>
+        </geometry>
+    </collision>
     </link>
     <gazebo reference="petal_five">
@@ -422,10 +366,10 @@
     	<child link="petal_six"/>
     	<axis xyz="0 0 1"/>
- 	<origin rpy="-0.2 0.2 0" xyz="-0.3 -0.3 0.05"/>
+ 	<origin rpy="-0.3 0.3 0" xyz="-0.3 -0.3 0.08"/>
     </joint>
     <link name="petal_six">
     <visual>
         <geometry>
-            <cylinder radius="${petal_radius}" length="${petal_height}"/> <!-- Измените параметры, если необходимо -->
+            <cylinder radius="${petal_radius}" length="${petal_height/4}"/> <!-- Измените параметры, если необходимо -->
         </geometry>
         <material name="orange"/>
@@ -433,15 +377,7 @@
     <collision>
         <geometry>
-            <cylinder radius="${petal_radius}" length="${petal_height}"/>
-        </geometry>
-    </collision>
-    <inertial>
-        <!-- Параметры инерции для stem -->
-        <origin xyz="0 0 0.05" rpy="0 0 0"/>
-        <mass value="0" />
-        <inertia ixx="1e-6" ixy="0.0" ixz="0.0"
-                 iyy="1e-6" iyz="0.0"
-                 izz="1e-6" />
-    </inertial>
+            <cylinder radius="${petal_radius}" length="${petal_height/4}"/>
+        </geometry>
+    </collision>
     </link>
     <gazebo reference="petal_six">
@@ -453,10 +389,10 @@
     	<child link="petal_seven"/>
     	<axis xyz="0 0 1"/>
- 	<origin rpy="-0.2 -0.2 0" xyz="0.3 -0.3 0.05"/>
+ 	<origin rpy="-0.3 -0.3 0" xyz="0.3 -0.3 0.08"/>
     </joint>
     <link name="petal_seven">
     <visual>
         <geometry>
-            <cylinder radius="${petal_radius}" length="${petal_height}"/> <!-- Измените параметры, если необходимо -->
+            <cylinder radius="${petal_radius}" length="${petal_height/4}"/> <!-- Измените параметры, если необходимо -->
         </geometry>
         <material name="orange"/>
@@ -464,15 +400,7 @@
     <collision>
         <geometry>
-            <cylinder radius="${petal_radius}" length="${petal_height}"/>
-        </geometry>
-    </collision>
-    <inertial>
-        <!-- Параметры инерции для stem -->
-        <origin xyz="0 0 0.05" rpy="0 0 0"/>
-        <mass value="0" />
-        <inertia ixx="1e-6" ixy="0.0" ixz="0.0"
-                 iyy="1e-6" iyz="0.0"
-                 izz="1e-6" />
-    </inertial>
+            <cylinder radius="${petal_radius}" length="${petal_height/4}"/>
+        </geometry>
+    </collision>
     </link>
     <gazebo reference="petal_seven">
@@ -484,10 +412,10 @@
     	<child link="petal_eight"/>
     	<axis xyz="0 0 1"/>
- 	<origin rpy="0.2 0.2 0" xyz="-0.3 0.3 0.05"/>
+ 	<origin rpy="0.3 0.3 0" xyz="-0.3 0.3 0.08"/>
     </joint>
     <link name="petal_eight">
     <visual>
         <geometry>
-            <cylinder radius="${petal_radius}" length="${petal_height}"/> <!-- Измените параметры, если необходимо -->
+            <cylinder radius="${petal_radius}" length="${petal_height/4}"/> <!-- Измените параметры, если необходимо -->
         </geometry>
         <material name="orange"/>
@@ -495,15 +423,7 @@
     <collision>
         <geometry>
-            <cylinder radius="${petal_radius}" length="${petal_height}"/>
-        </geometry>
-    </collision>
-    <inertial>
-        <!-- Параметры инерции для stem -->
-        <origin xyz="0 0 0.05" rpy="0 0 0"/>
-        <mass value="0" />
-        <inertia ixx="1e-6" ixy="0.0" ixz="0.0"
-                 iyy="1e-6" iyz="0.0"
-                 izz="1e-6" />
-    </inertial>
+            <cylinder radius="${petal_radius}" length="${petal_height/4}"/>
+        </geometry>
+    </collision>
     </link>
     <gazebo reference="petal_eight">
